Commit message: Add Echo robot model visualization launch

File: echo_workspace/src/echo_description/urdf/robots/mecanum.urdf.xacro (robot description, xacro)
@@ -9,4 +9,6 @@
   <xacro:include filename="$(find echo_description)/urdf/sensors/depth_sensor.urdf.xacro" />
   <xacro:include filename="$(find echo_description)/urdf/controllers/omni_drive.urdf.xacro" />
+  <xacro:property name="base_mesh_file" value="package://echo_description/meshes/base.dae" />
+  <xacro:property name="wheel_mesh_file" value="package://echo_description/meshes/tire.dae" />
   <xacro:base
     length="${base_length}"
